File: Taiplit20-pcb/Taiplit20-pcb.kicad_sch (KiCad schematic)
At the start: 0 parts

Commit message: Right PCB added
Parts:
- added BT1: Battery, Connector_JST:JST_PH_S2B-PH-K_1x02_P2.00mm_Horizontal, symbol Device:Battery
- added C1, C2: 1u, Capacitor_SMD:C_0603_1608Metric, symbol Device:C_Small
- added C3, C4: 100n, Capacitor_SMD:C_0603_1608Metric, symbol Device:C_Small
- added C5, C6, C7: 4u7, Capacitor_SMD:C_0603_1608Metric, symbol Device:C_Small
- added CH1, CH10, CH2, CH3, CH4, CH5, CH6, CH7, CH8, CH9: choc_v1_SW_HS, marbastlib-xp-choc:SW_choc_v2_HS_CPG135001S30_1u, symbol marbastlib-choc:choc_v1_SW_HS_CPG135001S30
- added D1, D10, D2, D3, D4, D5, D6, D7, D8, D9: D, Diode_SMD:D_SOD-123, symbol Device:D_Small
- added D11: BSD3C051V, Diode_SMD:D_SOD-323, symbol Device:D_TVS_Small
- added F1: 750mA, Fuse:Fuse_1206_3216Metric, symbol Device:Fuse_Small
- added J1: USB_C_Receptacle_USB2.0_16P, Connector_USB:USB_C_Receptacle_HRO_TYPE-C-31-M-12, symbol Connector:USB_C_Receptacle_USB2.0_16P
- added J2: Conn_ARM_JTAG_SWD_10, Connector_PinHeader_1.27mm:PinHeader_2x05_P1.27mm_Vertical, symbol Connector:Conn_ARM_JTAG_SWD_10
- added L1, L2: BLM15PX121SN1D, Inductor_SMD:L_0402_1005Metric, symbol Device:L_Small
- added LED1: Orange, LED_SMD:LED_0805_2012Metric, symbol Device:LED_Small
- added Q1: 2N7002, Package_TO_SOT_SMD:SOT-23, symbol Transistor_FET:2N7002
- added R1, R2: 5k1, Resistor_SMD:R_0603_1608Metric, symbol Device:R_Small
- added R10: 806k, Resistor_SMD:R_0603_1608Metric, symbol Device:R_Small
- added R11: 2M, Resistor_SMD:R_0603_1608Metric, symbol Device:R_Small
- added R3: 3k9, Resistor_SMD:R_0603_1608Metric, symbol Device:R_Small
- added R4, R6: 1k5, Resistor_SMD:R_0603_1608Metric, symbol Device:R_Small
- added R5, R9: 10k, Resistor_SMD:R_0603_1608Metric, symbol Device:R_Small
- added R7: 100k, Resistor_SMD:R_0603_1608Metric, symbol Device:R_Small
- added R8: 100R, Resistor_SMD:R_0603_1608Metric, symbol Device:R_Small
- added SW1: SW_RST, Button_Switch_SMD:SW_SPST_TL3342, symbol Switch:SW_Push
- added SW2: SW_SPDT, Button_Switch_SMD:SW_SPDT_CK_JS102011SAQN, symbol Switch:SW_SPDT
- added U1: nRF52840_holyiot_18010, marbastlib-various:nRF52840_holyiot_18010_HS_simple, symbol marbastlib-various:nRF52840_holyiot_18010
- added U2: XC6206PxxxMR, Package_TO_SOT_SMD:SOT-23-3, symbol Regulator_Linear:XC6206PxxxMR
- added U3: SRV05-4, Package_TO_SOT_SMD:SOT-23-6, symbol Power_Protection:SRV05-4
- added U4: BQ24075RGT, Package_DFN_QFN:VQFN-16-1EP_3x3mm_P0.5mm_EP1.6x1.6mm, symbol Battery_Management:BQ24075RGT
Connections:
- new net: CH4.2, D4.2 (A)
- new net: CH2.2, D2.2 (A)
- new net: LED1.1 (K), R6.1
- new net: R6.2, U4.9 (~{CHG})
- new net: CH5.2, D5.2 (A)
- new net: R7.2, SW2.1 (A)
- new net: CH3.2, D3.2 (A)
- new net: R5.1, U4.1 (TS)
- new net: R4.1, U4.12 (ILIM)
- new net: R3.1, U4.16 (ISET)
- new net: F1.1, L1.2
- new net: CH10.2, D10.2 (A)
- new net: CH6.2, D6.2 (A)
- new net: Q1.1 (G), R8.2, R9.1
- new net: CH8.2, D8.2 (A)
- new net: CH1.2, D1.2 (A)
- new net: CH9.2, D9.2 (A)
- new net: J1.A5 (CC1), R2.2
- new net: J1.B5 (CC2), R1.1
- new net: CH7.2, D7.2 (A)
- new net +3.3V: C2.1, C3.1, J2.1 (VTref), U1.14 (VDD_nRF), U2.2 (VO)
- new net +5V: C5.1, F1.2, R8.1, U1.22 (VBUS), U3.5 (VP), U4.13 (IN)
- new net +BATT: BT1.1 (+), C7.1, R7.1, U4.2 (BAT), U4.3 (BAT)
- new net +VSW: C1.1, C6.1, LED1.2 (A), R10.1, U2.3 (VI), U4.10 (OUT), U4.11 (OUT), U4.6 (EN1)
- new net Earth: C4.2, D11.1 (A1), J1.A1 (GND), J1.A12 (GND), J1.B1 (GND), J1.B12 (GND), J1.SH (SHIELD), L2.1
- new net GND: BT1.2 (-), C1.2, C2.2, C3.2, C4.1, C5.2, C6.2, C7.2, D11.2 (A2), J2.3 (GND), J2.5 (GND), J2.9 (GNDDetect), L2.2, Q1.2 (S), R1.2, R11.2, R2.1, R3.2, R4.2, R5.2, R9.2, SW1.2, SW2.3 (C), U1.1 (GND), U1.25 (GND), U1.37 (GND), U2.1 (GND), U3.2 (VN), U4.17 (VSS), U4.4 (~{CE}), U4.5 (EN2), U4.8 (VSS)
- new net RST: J2.10 (~{RESET}), SW1.1, U1.21 (P0.18-RESET)
- new net SWDCLK: J2.4 (SWCLK/TCK), U1.31 (SWDCLK)
- new net SWDIO: J2.2 (SWDIO/TMS), U1.32 (SWDIO)
- new net SYSOFF: Q1.3 (D), SW2.2 (B), U4.15 (SYSOFF)
- new net USB-D+: J1.A6 (D+), J1.B6 (D+), U1.24 (D+), U3.1 (IO1)
- new net USB-D-: J1.A7 (D-), J1.B7 (D-), U1.23 (D-), U3.6 (IO4)
- new net VBUS: J1.A4 (VBUS), J1.A9 (VBUS), J1.B4 (VBUS), J1.B9 (VBUS), L1.1
- new net VSENSE: R10.2, R11.1, U1.11 (P0.31-LF-A)
- new net col0: CH1.1, CH3.1, CH4.1, U1.10 (P0.30-LF-A)
- new net col1: CH2.1, CH5.1, CH6.1, U1.9 (P0.29-LF-A)
- new net col2: CH7.1, CH8.1, U1.8 (P0.28-LF-A)
- new net col3: CH10.1, CH9.1, U1.7 (P0.02-LF-A)
- new net row0: D3.1 (K), D5.1 (K), D7.1 (K), D9.1 (K), U1.15 (P0.07)
- new net row1: D10.1 (K), D4.1 (K), D6.1 (K), D8.1 (K), U1.16 (P1.09)
- new net row2: D1.1 (K), D2.1 (K), U1.17 (P0.12)
- no-connect marks 0 -> 45
